Commit message: FIX: fix ros planar move plugin bug

File: src/mecanum_robot_description/urdf/mecanum_robot_custom_control/mecanum.gazebo.xacro (robot description, xacro)
@@ -13,5 +13,5 @@
   </gazebo>
   <gazebo>
-    <plugin name="$custom_controller" filename="libropod_control_plugin.so">
+    <plugin name="$custom_controller" filename="libcustom_control_plugin.so">
         <commandTopic>/mecanum_vel</commandTopic>
         <odometryTopic>/odom</odometryTopic>

File: src/mecanum_robot_description/urdf/mecanum_robot_velodyne/mecanum.gazebo.xacro (robot description, xacro)
@@ -12,15 +12,13 @@
     <material>Gazebo/White</material>
   </gazebo>
-	<gazebo>
-	    <plugin name="omni_steering" filename="libgazebo_ros_planar_move.so">
-	      <commandTopic>mecanum_vel</commandTopic>
-	      <odometryTopic>odom</odometryTopic>
-	      <odometryFrame>odom</odometryFrame>
-	      <odometryRate>50.0</odometryRate>
-	      <robotBaseFrame>base_footprint</robotBaseFrame>
-	      <publishTF>true</publishTF>
-	    </plugin>
-		<material>Gazebo/DarkGrey</material>
-	</gazebo>
+  <gazebo>
+    <plugin name="$custom_controller" filename="libcustom_control_plugin.so">
+        <commandTopic>/mecanum_vel</commandTopic>
+        <odometryTopic>/odom</odometryTopic>
+        <odometryFrame>/odom</odometryFrame>
+        <odometryRate>20.0</odometryRate>
+        <robotBaseFrame>/mecanum/base_link</robotBaseFrame>
+    </plugin>
+</gazebo>
   </xacro:macro>
   <xacro:macro name="sensor_gazebo" params="">
