Commit message: EDIT: mecanum model urdf

File: src/mecanum_robot_description/urdf/mecanum_robot_custom_control/cycloid_gear_mecanum_wheel.urdf.xacro (robot description, xacro)
@@ -11,5 +11,5 @@
         <xacro:property name="radius" value="0.0762"/>
         <xacro:property name="length" value="0.045"/>
-        <joint name="${prefix}_wheel_joint" type="continuous">
+        <joint name="${prefix}_wheel_joint" type="continuous"> <!--fixed!-->
             <parent link="${parent}"/>
             <child link="${prefix}_wheel"/>
@@ -71,10 +71,10 @@
         </transmission>
         <gazebo reference="${prefix}_wheel">
-            <mu1>1.0</mu1>
-            <mu2>1.0</mu2>
+            <mu1>0.0</mu1>
+            <mu2>0.0</mu2>
             <kp>1e+13</kp>
             <kd>1.0</kd>
             <!-- <maxVel>0.001</maxVel> -->
-            <!-- <minDepth>0.00000000001</minDepth> -->
+            <minDepth>0.001</minDepth>
             <!-- <turnGravityOff>true</turnGravityOff> -->
             <!-- <gravity>1</gravity> -->

File: src/mecanum_robot_description/urdf/mecanum_robot_custom_control/mecanum.gazebo.xacro (robot description, xacro)
@@ -28,5 +28,5 @@
       <controlPeriod>1</controlPeriod>
       <robotNamespace>/mecanum</robotNamespace>
-      <!--jointName>front_R_wheel_joint, front_L_wheel_joint, back_R_wheel_joint, back_L_wheel_joint </jointName-->
+      <!-- <jointName>front_R_wheel_joint, front_L_wheel_joint, back_R_wheel_joint, back_L_wheel_joint </jointName> -->
       <robotSimType>gazebo_ros_control/DefaultRobotHWSim</robotSimType>
       <!--legacyModeNS>true</legacyModeNS-->
